Commit message: Practical 4

File: src/my_r2d2/urdf/r2d2.urdf (robot description, URDF)
Before this commit: robot r2d2, 16 links, 15 joints
Links:
- added link base_footprint
- added link lense, mass 0.05; collision sphere radius=0.035; visual sphere radius=0.035
Joints:
- added joint base_footprint_joint: type fixed, parent base_link, child base_footprint, origin xyz=0 0 -0.47
- added joint lense_joint: type prismatic, parent box, child lense, origin xyz=-0.015 0 0 rpy=0 0 0, limit lower=-0.035 upper=0 effort=1000.0 velocity=0.5

File: src/my_r2d2/urdf/r2d2.urdf.xacro (robot description, xacro)
@@ -366,3 +366,10 @@
     <origin rpy="0 0 0" xyz="-0.015 0 0"/>
   </joint>
+  <link name="base_footprint">
+  </link>
+  <joint name="base_footprint_joint" type="fixed">
+    <parent link="base_footprint"/>
+    <child link="base_link"/>
+    <origin xyz="0 0 0.47"/>
+  </joint>
 </robot>
