Commit message: practical 5

File: src/my_r2d2/urdf/r2d2.urdf.xacro (robot description, xacro)
@@ -373,3 +373,10 @@
     <origin xyz="0 0 0.47"/>
   </joint>
+  <link name="eye">
+  </link>
+  <joint name="lense_to_eye" type="fixed">
+      <parent link="lense"/>
+      <child link="eye"/>
+      <origin rpy="${pi/2} ${pi}  ${pi/2}"/>
+  </joint>
 </robot>
